File: MLX90632_rigid.kicad_sch (KiCad schematic)
At the start: 5 parts, among them U1 MLX90632SLD-DCB-000-RE

Commit message: Update for Ver2.0
Parts:
- FPC1: value ~ -> (none)
- R1, R2: footprint Resistor_SMD:R_0603_1608Metric -> Resistor_SMD:R_0402_1005Metric
